File: Schematic/Schematic.kicad_sch (KiCad schematic)
At the start: 0 parts

Commit message: initial peripheral connections and downloaded libraries
Parts:
- added BT1: 5000 maH LiPo, symbol Aerothon_Custom:GNB_5000mah_6S
- added C1: Arducam, symbol Aerothon_Custom:Arducam
- added C2: FPV Cam, symbol Aerothon_Custom:FPV
- added C3: 1000uF 35V, EEUFR1E102:CAPPRD500W60D1000H2000, symbol EEUFR1E102:EEUFR1E102
- added C4: 470uF 25V Low ESR, symbol Device:C
- added C5: 0.1uF Ceramic, symbol Device:C
- added E1: ESC, symbol Aerothon_Custom:ESC
- added J1: XT60-M, XT60-M:AMASS_XT60-M, symbol XT60-M:XT60-M
- added L1: 100uH, symbol Device:L
- added M1, M2, M3, M4: (no value), symbol Aerothon_Custom:Motors
- added T1: Telemetry, symbol Aerothon_Custom:3DR_Telemetry
- added U1: Matek PDB, symbol Aerothon_Custom:Matek
- added U2: DRV8838, Package_SON:WSON-8-1EP_2x2mm_P0.5mm_EP0.9x1.6mm, symbol Driver_Motor:DRV8838
Connections:
- new net: E1. (M1), M2.1 (A), M2.2 (B), M2.3 (C)
- new net: E1. (M1), M3.1 (A), M3.2 (B), M3.3 (C)
- new net: E1. (M1), M4.1 (A), M4.2 (B), M4.3 (C)
- new net: E1. (M1), M1.1 (A), M1.2 (B), M1.3 (C)
- new net: C4.2, C5.1
- new net 10V: U1.4 (10V_OUT)
- new net 3V3: C1.22 (CAM_3v3), U2.7 (~{SLEEP})
- new net 5V: L1.1, T1.1 (VCC), U1.3 (5V_OUT), U2.8 (VCC)
- new net CURR: U1.13 (CURR)
- new net CURR_SENSE: E1.7 (CRT)
- new net FPV_5V: C2.1 (5V), C4.1, L1.2
- new net GND: BT1.1 (GND), C1.1 (GND), C1.10 (GND), C1.13 (GND), C1.16 (GND), C1.19 (GND), C1.4 (GND), C1.7 (GND), C2.2 (GND), C3.N, C5.2, E1. (M1), E1.6 (GND), E1.9 (GND), J1.N (NEG), T1.6 (GND), U1.2 (GND), U2.4 (GND), U2.9 (GND)
- new net PWM1: E1.4 (S1)
- new net PWM2: E1.3 (S2)
- new net PWM3: E1.2 (S3)
- new net PWM4: E1.1 (S4)
- new net TELEM_RX: T1.RX (3)
- new net TELEM_TX: T1.TX (2)
- new net VBAT_SENSE: E1.8 (BAT)
- new net VBat: BT1.8 (Vbat), J1.P (POS)
- new net Vbat: C3.P, E1. (M1), U1.1 (BAT+)
- no-connect marks 0 -> 16

Commit message: cleanup
Parts:
- added O1: (no value), symbol Aerothon_Custom:Oak-d-lite
Changed lines of the file:
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@@
+	)
+	(symbol
+		(lib_id "Aerothon_Custom:Oak-d-lite")
+		(at 81.28 110.49 0)
+		(unit 1)
+		(body_style 1)
+		(exclude_from_sim no)
+		(in_bom yes)
+		(on_board yes)
+		(in_pos_files yes)
+		(dnp no)
+		(fields_autoplaced yes)
+		(property "Reference" "O1"
+			(at 81.915 105.41 0)
+			(show_name no)
+			(do_not_autoplace no)
+			(effects
+				(font
+					(size 1.27 1.27)
+				)
+			)
+		)
+		(property "Value" ""
+			(at 81.28 110.49 0)
+			(show_name no)
+			(do_not_autoplace no)
+			(effects
+				(font
+					(size 1.27 1.27)
+				)
+			)
+		)
+		(property "Footprint" ""
+			(at 81.28 110.49 0)
+			(hide yes)
+			(show_name no)
+			(do_not_autoplace no)
+			(effects
+				(font
+					(size 1.27 1.27)
+				)
+			)
+		)
+		(property "Datasheet" ""
+			(at 81.28 110.49 0)
+			(hide yes)
+			(show_name no)
+			(do_not_autoplace no)
+			(effects
+				(font
+					(size 1.27 1.27)
+				)
+			)
+		)
+		(property "Description" ""
+			(at 81.28 110.49 0)
+			(hide yes)
+			(show_name no)
+			(do_not_autoplace no)
+			(effects
+				(font
+					(size 1.27 1.27)
+				)
+			)
+		)
+		(pin "1"
+		)
+		(pin "10"
+		)
+		(instances
+			(project "Schematic"
+				(path "/5c69f783-11c5-4401-9233-9a1d77a80e45"
+					(reference "O1")
+					(unit 1)
+				)
+			)
+		)
 	)
 	(symbol

Commit message: 6x and Jetson schematic
Parts:
- added J2: Header, symbol Connector:DIN41612_02x10_AB
- added J3: Barrel_Jack_Switch, symbol Connector:Barrel_Jack_Switch
- added M5: N20 Geared Motor, symbol Motor:Motor_DC
- added U3: (no value), symbol Aerothon_custom-2:Pixahawk_6X_Mini_baseboard
- added U4: (no value), symbol Aerothon_custom-2:Skydroid R12
- added U5: (no value), symbol Aerothon_custom-2:Jetson_Nano
Connections:
- net 10V: now also J3.1
- net 3V3: now also J2. (Pin_b10)
- net 5V: now also J2. (Pin_b10)
- net GND: now also J2. (Pin_b10), J3.2, U4. (2.4G_ANT)
- net at U2.2 (OUT1): now also M5.1 (+)
- net at U2.3 (OUT2): now also M5.2 (-)
- new net 1V8: J2. (Pin_b10)
- new net AUTO_PWR: J2. (Pin_b10)
- new net CAN0: J2. (Pin_b10)
- new net CAN1: J2. (Pin_b10)
- new net GPIO: J2. (Pin_b10)
- new net SPI: J2. (Pin_b10)
- new net UART0: J2. (Pin_b10)
- new net UART1: J2. (Pin_b10)
- no-connect marks 16 -> 19
Other:
- note added: "USB Splitter"
- moved on the sheet: BT1, C1, C2, C3, C4, C5, E1, J1, L1, M1, M2, M3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
